Commit message: Update joint limits

File: Kinematics/robot.urdf (robot description, URDF)
Before this commit: robot robot, 9 links, 8 joints
Joints:
- joint joint0: limit lower=-1.8 upper=1.8 effort=10.0 velocity=3.14159265 -> lower=-2.268928 upper=2.268928 effort=10.0 velocity=3.14159265
- joint joint1: limit lower=-1.8 upper=1.8 effort=10.0 velocity=3.14159265 -> lower=-2.268928 upper=2.268928 effort=10.0 velocity=3.14159265
- joint joint2: limit lower=-1.8 upper=1.8 effort=10.0 velocity=3.14159265 -> lower=-2.268928 upper=2.268928 effort=10.0 velocity=3.14159265
- joint joint3: limit lower=-1.8 upper=1.8 effort=10.0 velocity=3.14159265 -> lower=-2.268928 upper=2.268928 effort=10.0 velocity=3.14159265
- joint joint4: limit lower=-1.8 upper=1.8 effort=10.0 velocity=3.14159265 -> lower=-2.268928 upper=2.268928 effort=10.0 velocity=3.14159265
- joint joint5: limit lower=-3 upper=3 effort=10.0 velocity=3.14159265 -> lower=-3.14 upper=3.14 effort=10.0 velocity=3.14159265
